Commit message: Added cardboard box

File: models/openarm_mujoco.urdf (robot description, URDF)
Before this commit: robot openarm_v20, 22 links, 21 joints
Joints:
- joint openarm_left_finger_joint1: limit lower=-1.5708 upper=0 effort=7 velocity=5 -> lower=-0.80 upper=0 effort=7 velocity=5
- joint openarm_left_finger_joint2: limit lower=0 upper=1.5708 effort=7 velocity=5 -> lower=0 upper=0.80 effort=7 velocity=5
- joint openarm_right_finger_joint1: limit lower=-1.5708 upper=0 effort=7 velocity=5 -> lower=-0.80 upper=0 effort=7 velocity=5
- joint openarm_right_finger_joint2: limit lower=0 upper=1.5708 effort=7 velocity=5 -> lower=0 upper=0.80 effort=7 velocity=5
